Commit message: extend_length = 0.06 要提交的变更： 	修改：     src/ur5_grasping_demo/ur5_arm_description/urdf/ur5.gv 	修改：     src/ur5_grasping_demo/ur5_arm_description/urdf/ur5.pdf 	修改：     src/ur5_grasping_demo/ur5_arm_description/urdf/ur5_robot.urdf 	修改：     src/ur5_grasping_demo/ur5_arm_description/urdf/ur5_robot.urdf.xacro 	修改：     src/ur5_grasping_demo/ur5_arm_moveit_config/.setup_assistant 	修改：     src/ur5_grasping_demo/ur5_arm_moveit_config/config/ur5.srdf 	修改：     src/ur5_grasping_demo/ur5_arm_moveit_config/package.xml

File: src/ur5_grasping_demo/ur5_arm_description/urdf/ur5_robot.urdf (robot description, URDF)
Before this commit: robot ur5, 26 links, 25 joints
Joints:
- joint wrist_3_link-tool0_fixed_joint: origin xyz=0 0.0923 0 rpy=-1.5707963267948966 0 0 -> xyz=0 0.14229999999999998 0 rpy=-1.5707963267948966 0 0

File: src/ur5_grasping_demo/ur5_arm_description/urdf/ur5_robot.urdf.xacro (robot description, xacro)
@@ -7,5 +7,5 @@
     <xacro:include filename="$(find ur_description)/urdf/ur5.urdf.xacro" />
     <!-- 加载arm,相当于前面是函数，下面这个是引用-->
-    <xacro:ur5_robot prefix="" joint_limited="false" extend_length="0.01"/>
+    <xacro:ur5_robot prefix="" joint_limited="false" extend_length="0.06"/>
     <!-- robotiq 85 -->
     <xacro:include filename="$(find robotiq_85_description)/urdf/robotiq_85_gripper.urdf.xacro" />
